File: smart-wakeup-pcb/smart-wakeup-pcb.kicad_sch (KiCad schematic)
At the start: 21 parts, among them J1 Conn_01x03, J2 Conn_01x02, J3 Conn_01x04, J4 Conn_01x04, J5 Conn_01x02, J6 Conn_01x02, Q1 BSS138, Q2 BSS138, U1 XIAO-ESP32-S3-SMD, U2 MAX98357A

Commit message: reroute
Parts:
- added C4: 0.1u, Capacitor_SMD:C_0603_1608Metric, symbol Device:C_Small
- added U3: TMP102xxDRL, Package_TO_SOT_SMD:SOT-563, symbol Sensor_Temperature:TMP102xxDRL
- J1: footprint Connector_JST:JST_PH_B3B-PH-K_1x03_P2.00mm_Vertical -> Connector_JST:JST_PH_S3B-PH-K_1x03_P2.00mm_Horizontal
- J2: footprint Connector_JST:JST_PH_B2B-PH-K_1x02_P2.00mm_Vertical -> Connector_JST:JST_PH_S2B-PH-K_1x02_P2.00mm_Horizontal
- J4: footprint Connector_JST:JST_PH_B4B-PH-K_1x04_P2.00mm_Vertical -> Connector_JST:JST_PH_S4B-PH-K_1x04_P2.00mm_Horizontal
- R1, R2, R3, R4: value R -> 10k; footprint Capacitor_SMD:C_0603_1608Metric -> Resistor_SMD:R_0603_1608Metric
Connections:
- net +3.3V: now also C4.1, U3.5 (V+)
- net GND: now also C4.2, U3.2 (GND), U3.4 (ADD0)
- net I2C_SCL_3V3: now also U1.10 (PA5_A9_D9_MISO), U3.1 (SCL); no longer U1.6 (PA9_A5_D5_SCL)
- net I2C_SDA_3V3: now also U1.9 (PA7_A8_D8_SCK), U3.6 (SDA); no longer U1.5 (PA8_A4_D4_SDA)
- net I2S_BCLK: now also U1.5 (PA8_A4_D4_SDA); no longer U1.10 (PA5_A9_D9_MISO)
- net I2S_DIN: now also U1.6 (PA9_A5_D5_SCL); no longer U1.11 (PA6_A10_D10_MOSI)
- net I2S_LRCLK: now also U1.3 (PA10_A2_D2); no longer U1.9 (PA7_A8_D8_SCK)
- net SW_1_IN: now also U1.11 (PA6_A10_D10_MOSI); no longer U1.7 (PB08_A6_D6_TX)
- no-connect marks 0 -> 3
Other:
- moved on the sheet: J1, Q2, R3, R4

Commit message: drc, holes, lux sensor
Parts:
- added C5: 1u, Capacitor_SMD:C_0603_1608Metric, symbol Device:C_Small
- added H1, H2: MountingHole, MountingHole:MountingHole_2.2mm_M2, symbol Mechanical:MountingHole
- added U4: LTR-303ALS-01, OptoDevice:Lite-On_LTR-303ALS-01, symbol Sensor_Optical:LTR-303ALS-01
Connections:
- net +3.3V: now also C5.1, U4.1 (VDD)
- net +5V: no longer U1.14 (5V)
- net GND: now also C5.2, U4.3 (GND)
- net I2C_SCL_3V3: now also U4.4 (SCL)
- net I2C_SDA_3V3: now also U4.6 (SDA)
- no-connect marks 3 -> 5

Commit message: labeling and test points
Parts:
- added J10: Conn_01x03, Connector_PinHeader_1.00mm:PinHeader_1x03_P1.00mm_Vertical, symbol Connector_Generic:Conn_01x03
- added J7: Conn_01x06, Connector_PinHeader_1.00mm:PinHeader_1x06_P1.00mm_Vertical, symbol Connector_Generic:Conn_01x06
- added J9: Conn_01x04, Connector_PinHeader_1.00mm:PinHeader_1x04_P1.00mm_Vertical, symbol Connector_Generic:Conn_01x04
- added TP1, TP2, TP3: TestPoint, TestPoint:TestPoint_Pad_D1.5mm, symbol Connector:TestPoint
Connections:
- net +3.3V: now also J7.4 (Pin_4)
- net GND: now also J10.2 (Pin_2), J7.1 (Pin_1), J9.2 (Pin_2), TP3.1
- net I2C_SCL: now also TP2.1
- net I2C_SCL_3V3: now also J7.3 (Pin_3)
- net I2C_SDA: now also TP1.1
- net I2C_SDA_3V3: now also J7.2 (Pin_2)
- net I2S_BCLK: now also J7.6 (Pin_6)
- net I2S_DIN: now also J9.1 (Pin_1)
- net I2S_LRCLK: now also J7.5 (Pin_5)
- net SW_1_IN: now also J10.1 (Pin_1)
- net SW_2_IN: now also J10.3 (Pin_3)
- net SPKR_N: now reaches J2.2 (Pin_2), U2.10 (OUTN)
- net SPKR_N: now also J9.4 (Pin_4)
- net SPKR_P: now reaches J2.1 (Pin_1), U2.9 (OUTP)
- net SPKR_P: now also J9.3 (Pin_3)
